File: PCB/Boom-1/Boom-1.kicad_pcb (KiCad board)
At the start: 2 copper layers, 698 parts, among them J1 NoiseIOConn, J10 Osc1HFTrackConn, J11 Osc1FiltCVConn, J12 OscFiltEnv1Conn, J13 OscFiltEnv2Conn, J14 SubFiltEnv1Conn, J15 SubFiltEnv2Conn, J16 Osc1FXConn, J17 SubFXConn, J18 Osc1FiltCVConn, J19 Osc1FiltCVConn, J2 Osc2CVConn, J20 Osc2FXConn, J21 OscAmpEnvConn, J22 SubAmpEnvConn, J23 OscAmpEnvBypass, J24 SubAmpAudioBypass, J25 SubAmpEnvBypass, J26 PreFV1FXConn, J27 PowerConn, J28 FV1Conn, J29 IOConn, J3 Osc1CVConn, J4 Osc2SyncConn, J5 Osc1SyncConn, J6 Osc2ScaleConn, J7 Osc2HFTrackConn, J8 SubIOConn, J9 Osc1ScaleConn, Q1 2N3904, SW1 SW_DIP_x04, U1 CEM3340, U10 AS3320, U11 AS3310, U12 AS3310, U13 AS3310, U14 AS3310, U15 V2164D, U16 AS3310, U17 AS3310, U18 V2164D, U19 TL074, U2 CEM3340, U20 TL074, U21 TL074, U22 TL074, U23 TL074, U24 TL074, U25 TL074, U26 TL074, U27 TL072, U28 TL074, U29 TL072, U3 4013, U30 TL074, U31 TL072, U32 TL074, U33 TL074, U34 TL074, U35 TL072, U36 TL074, U37 TL074, U38 TL072, U39 TL074, U4 NOISE, U40 TL072, U41 TL074, U42 TL074, U43 TL074, U44 TL074, U45 L7905, U46 L7805, U5 V2164D, U6 V2164D, U7 V2164D, U8 AS3320, U9 AS3320

Commit message: misc
Parts:
- moved U7 784.6 mm to (-565.1, 152.1)
- moved U4 714.9 mm to (-623.6, 121.9)
- moved U25 502.0 mm to (-565.4, 123.7)
Changed lines of the file:
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@@
   )
   (module Package_DIP:DIP-8_W7.62mm_Socket (layer F.Cu)
-    (at 85.09 27.94)
+    (at -623.57 121.92)
     (descr "8-lead though-hole mounted DIP package, row spacing 7.62 mm (300 mils), Socket")
     (tags "THT DIP DIL PDIP 2.54mm 7.62mm 300mil Socket")
@@
   )
   (module Package_DIP:DIP-16_W7.62mm_Socket (layer F.Cu)
-    (at 209.55 27.94)
+    (at -565.15 152.146)
     (descr "16-lead though-hole mounted DIP package, row spacing 7.62 mm (300 mils), Socket")
     (tags "THT DIP DIL PDIP 2.54mm 7.62mm 300mil Socket")
@@
   )
   (module Package_DIP:DIP-14_W7.62mm (layer F.Cu)
-    (at -68.58 195.58)
+    (at -565.404 123.698)
     (descr "14-lead though-hole mounted DIP package, row spacing 7.62 mm (300 mils)")
     (tags "THT DIP DIL PDIP 2.54mm 7.62mm 300mil")

Commit message: gathered parts for subosc
Parts:
- moved TP1 1017.7 mm to (-673.6, 26.9)
- moved C3 985.4 mm to (-673.4, 37.6), turned to 270 degrees
- moved R1 933.9 mm to (-673.4, 46.0)
- moved TP5 921.0 mm to (-597.4, 18.8)
- moved C20 918.3 mm to (-577.3, 10.4)
- moved C14 917.7 mm to (-645.9, 28.2), turned to 90 degrees
- moved R23 909.6 mm to (-636.8, 33.8), turned to 270 degrees
- moved C31 903.3 mm to (-585.2, 56.6)
- moved C7 896.2 mm to (-619.8, 25.4)
- moved R9 891.2 mm to (-648.5, 18.0), turned to 180 degrees
- moved C48 887.2 mm to (-501.9, -81.0)
- moved R20 886.5 mm to (-631.7, 38.9)
- moved R106 884.8 mm to (-579.9, 4.83)
- moved TP3 883.7 mm to (-588.0, 45.7)
- moved C21 880.1 mm to (-557.5, 10.4)
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
Commit message: gathered components for noise
Parts:
- moved C30 963.2 mm to (-661.7, 177.3), turned to 180 degrees
- moved C45 936.7 mm to (-630.4, 222.5), turned to 180 degrees
- moved TP6 932.7 mm to (-602.0, 183.4)
- moved C26 930.5 mm to (-670.8, 187.5)
- moved TP25 925.8 mm to (-612.6, 226.6)
- moved C39 925.3 mm to (-602.0, 216.7)
- moved C44 917.5 mm to (-636.3, 209.6), turned to 270 degrees
- moved TP7 911.2 mm to (-605.3, 152.1)
- moved R121 906.1 mm to (-630.9, 202.2), turned to 90 degrees
- moved C35 902.5 mm to (-602.0, 165.9)
- moved C36 890.1 mm to (-602.2, 197.1)
- moved R21 886.6 mm to (-670.8, 182.4)
- moved R122 875.1 mm to (-615.7, 208.3), turned to 180 degrees
- moved R93 873.2 mm to (-623.8, 160.0)
- moved TP24 870.0 mm to (-616.2, 192.5)
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
Commit message: gathered components for osc1 filt 1
Parts:
- moved R190 894.4 mm to (-449.1, -269.7), turned to 180 degrees
- moved TP30 884.1 mm to (-315.5, -329.4)
- moved R170 883.7 mm to (-448.1, -262.4), turned to 180 degrees
- moved R169 868.2 mm to (-440.9, -265.9), turned to 270 degrees
- moved R224 857.9 mm to (-436.4, -270.3)
- moved C94 848.9 mm to (-324.4, -301.5)
- moved R146 834.3 mm to (-401.8, -258.3), turned to 180 degrees
- moved C90 833.1 mm to (-317.2, -299.0)
- moved C91 832.6 mm to (-296.2, -304.0)
- moved TP32 829.9 mm to (-288.0, -284.7)
- moved J18 828.0 mm to (-326.6, -275.3)
- moved R200 827.2 mm to (-334.8, -306.6)
- moved R154 827.2 mm to (-401.8, -261.6), turned to 180 degrees
- moved C108 826.0 mm to (-295.7, -284.7)
- moved C95 821.4 mm to (-295.9, -291.3)
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
Commit message: Gathered parts for osc2 filt 1
Parts:
- moved TP33 795.0 mm to (-368.8, -124.2)
- moved J19 787.0 mm to (-384.0, -83.1)
- moved TP28 786.7 mm to (-345.9, -137.7)
- moved C98 766.3 mm to (-372.9, -105.9)
- moved C93 745.5 mm to (-337.1, -108.2)
- moved R172 739.0 mm to (-380.2, -116.3)
- moved C102 726.6 mm to (-314.7, -111.8)
- moved R147 726.3 mm to (-387.1, -100.8)
- moved C96 724.6 mm to (-334.8, -116.8)
- moved TP31 722.7 mm to (-307.1, -96.8)
- moved C99 721.7 mm to (-354.1, -105.9)
- moved C97 719.0 mm to (-334.5, -112.5)
- moved R155 714.2 mm to (-387.1, -105.9)
- moved C92 713.4 mm to (-313.7, -116.8)
- moved C109 710.9 mm to (-313.7, -101.6)
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
Commit message: Gathered parts for subosc filt 1
Parts:
- moved C53 715.6 mm to (-384.0, 48.8)
- moved C80 701.2 mm to (-370.1, 59.7), turned to 90 degrees
- moved TP27 695.7 mm to (-341.4, 31.2)
- moved C79 692.1 mm to (-364.0, 41.4)
- moved J11 681.8 mm to (-371.3, 26.7), turned to 90 degrees
- moved C83 664.5 mm to (-315.5, 50.0)
- moved R143 664.0 mm to (-350.5, 37.3)
- moved TP29 663.1 mm to (-301.8, 66.5)
- moved R138 662.0 mm to (-357.9, 65.3)
- moved C59 656.2 mm to (-333.8, 50.5)
- moved R175 646.0 mm to (-319.5, 25.4), turned to 270 degrees
- moved J17 645.5 mm to (-348.5, 15.0), turned to 90 degrees
- moved C87 645.3 mm to (-308.4, 63.0)
- moved R158 644.5 mm to (-329.2, 37.6), turned to 90 degrees
- moved R219 635.4 mm to (-305.8, 58.2)
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
Commit message: gathered U components for remaining functional areas
Parts:
- moved C169 1356.4 mm to (-1018.8, 55.6)
- moved C154 1354.8 mm to (-1022.1, 5.08)
- moved C155 1354.4 mm to (-1018.5, 22.9)
- moved C168 1351.2 mm to (-1039.9, 55.6)
- moved C165 1350.6 mm to (-1020.3, 41.1)
- moved C153 1341.3 mm to (-1050.3, 18.5)
- moved C164 1337.0 mm to (-1046.7, 40.9)
- moved C152 1308.1 mm to (-1054.1, 4.57)
- moved J27 1087.9 mm to (-1067.1, -42.7)
- moved U46 1087.9 mm to (-1027.7, -16.0)
- moved U45 1087.9 mm to (-1048.0, -16.0)
- moved RV10 931.8 mm to (-525.5, -279.9)
- moved RV11 931.0 mm to (-522.2, -214.6)
- moved U27 811.9 mm to (-440.2, -280.7)
- moved U44 811.6 mm to (576.1, 45.0)
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
Commit message: updated from schematic
Connections:
- C64 pad 1: GND -> Net-(C64-Pad1)
- C95 pad 1: GND -> Net-(C95-Pad1)
- C96 pad 1: GND -> Net-(C96-Pad1)
- J29 pad 10: Net-(J29-Pad10) -> GND
- U10 pad 11: GND -> Net-(C64-Pad1)
- U8 pad 11: GND -> Net-(C95-Pad1)
- U9 pad 11: GND -> Net-(C96-Pad1)
