File: PCB/Boom-1/Boom-1.sch (KiCad schematic (older format))
At the start: 705 parts, among them J1 NoiseIOConn, J10 Osc1HFTrackConn, J11 SubFiltConn, J12 OscFiltEnv1Conn, J13 OscFiltEnv2Conn, J14 SubFiltEnv1Conn, J15 SubFiltEnv2Conn, J16 Osc1FiltConn, J17 OscFiltEnv1CVConn, J2 Conn_01x07, J20 Osc2FiltConn, J21 OscAmpEnvConn, J22 SubAmpEnvConn, J23 OscAmpEnvBypass, J24 SubAmpAudioBypass, J25 SubAmpEnvBypass, J26 PreFV1FXConn, J27 PowerConn, J28 FV1Conn, J29 IOConn, J3 Osc1CVConn, J4 Osc2SyncConn, J5 Osc1SyncConn, J6 Osc2ScaleConn, J7 Osc2HFTrackConn, J8 Conn_01x03, J9 Osc1ScaleConn, Q1 2N3904, SW1 SW_DIP_x04, U1 CEM3340, U10 AS3320, U11 AS3310, U12 AS3310, U13 AS3310, U14 AS3310, U15 V2164D, U16 AS3310, U17 AS3310, U18 V2164D, U19 TL074, U2 CEM3340, U20 TL074, U21 TL072, U22 TL074, U23 TL074, U24 TL072, U25 TL074, U26 TL074, U27 TL072, U28 TL074, U29 TL072, U3 4013, U30 TL072, U31 TL072, U32 TL074, U33 TL074, U34 TL074, U35 TL072, U36 TL074, U37 TL074, U38 TL072, U39 TL074, U4 NOISE, U40 TL072, U41 TL074, U42 TL074, U43 TL074, U44 TL074, U45 L7905, U46 L7805, U47 TL072, U48 TL072, U49 TL072, U5 V2164D, U6 V2164D, U7 V2164D, U8 AS3320, U9 AS3320

Commit message: filt env1 layout and routing DONE
Parts:
- removed RV10: 100K, Potentiometer_THT:Potentiometer_Piher_PT-6-V_Vertical, symbol Device:R_POT_TRIM_US
Connections:
- wire segments 3065 -> 3059
Changed lines of the file:
@@
 Wire Wire Line
 	41450 30050 42050 30050
-$Comp
-L Device:R_POT_TRIM_US RV10
-U 1 1 5FE55C96
-P 20450 17750
-F 0 "RV10" H 20382 17796 50  0000 R CNN
-F 1 "100K" H 20382 17705 50  0000 R CNN
-F 2 "Potentiometer_THT:Potentiometer_Piher_PT-6-V_Vertical" H 20450 17750 50  0001 C CNN
-F 3 "~" H 20450 17750 50  0001 C CNN
-	1    20450 17750
-	-1   0    0    1
-$EndComp
-Wire Wire Line
-	20450 17950 20450 17900
-Wire Wire Line
-	20450 17600 20450 17500
-$Comp
-L power:GND #PWR0124
-U 1 1 5FE55C81
-P 20450 17500
-F 0 "#PWR0124" H 20450 17250 50  0001 C CNN
-F 1 "GND" H 20455 17327 50  0000 C CNN
-F 2 "" H 20450 17500 50  0001 C CNN
-F 3 "" H 20450 17500 50  0001 C CNN
-	1    20450 17500
-	-1   0    0    1
-$EndComp
 Connection ~ 24950 21400
 Wire Wire Line
@@
 Connection ~ 20850 17950
 Wire Wire Line
-	20850 17950 20550 17950
-Wire Wire Line
 	22950 17850 21800 17850
 $Comp
@@
 	22050 15000 18300 15000
 Wire Wire Line
-	18300 15000 18300 17750
+	18300 15000 18300 17950
 Wire Wire Line
 	32850 27600 33650 27600
@@
 Wire Wire Line
 	19350 48200 20350 48200
-Wire Wire Line
-	20300 17750 20150 17750
 $Comp
 L Device:R_POT_TRIM_US RV11
@@
 Wire Wire Line
 	21150 20450 21150 20800
-Wire Wire Line
-	20150 17750 20150 18050
-Wire Wire Line
-	20150 18050 20450 18050
-Wire Wire Line
-	20450 18050 20450 20800
-Connection ~ 20150 17750
-Wire Wire Line
-	20550 17950 20550 20800
-Connection ~ 20550 17950
-Wire Wire Line
-	20550 17950 20450 17950
 $Comp
 L power:GND #PWR0122
@@
 Text Notes 20550 21100 3    50   ~ 0
 OscFiltEnv1AmtHigh
-Text Notes 20650 21100 3    50   ~ 0
-OscFiltEnv1Gate
 Text Notes 20750 21100 3    50   ~ 0
+OscFiltEnv1Gate
+Text Notes 20650 21100 3    50   ~ 0
 OscFiltEnv1Trigger
 Text Notes 20900 21100 3    50   ~ 0
@@
 	29350 37350 29350 43300
 Wire Wire Line
-	18300 17750 20150 17750
-Wire Wire Line
 	18600 24650 20250 24650
 Wire Wire Line
@@
 Connection ~ 18600 24650
 Wire Wire Line
-	18300 30050 18300 17750
+	18300 30050 18300 17950
 Wire Wire Line
 	18300 30050 22050 30050
-Connection ~ 18300 17750
+Connection ~ 18300 17950
 Wire Wire Line
 	28300 32100 28450 32100
@@
 AudioOutput
 Wire Wire Line
-	20650 19200 21450 19200
-Wire Wire Line
-	20650 19200 20650 20800
-Wire Wire Line
 	21450 19400 21400 19400
 Wire Wire Line
@@
 Connection ~ 22700 19800
 Wire Wire Line
-	20750 19700 22050 19700
-Wire Wire Line
-	20750 19700 20750 20800
-Wire Wire Line
 	21450 26300 21400 26300
 Wire Wire Line
@@
 	0    -1   1    0
 $EndComp
+Wire Wire Line
+	20650 20800 20650 19700
+Wire Wire Line
+	20650 19700 22050 19700
+Wire Wire Line
+	20450 17950 20450 20800
+Wire Wire Line
+	18300 17950 20450 17950
+Wire Wire Line
+	20750 20800 20750 19200
+Wire Wire Line
+	20750 19200 21450 19200
+Wire Wire Line
+	20550 20800 20550 17950
+Wire Wire Line
+	20550 17950 20850 17950
 $EndSCHEMATC

Commit message: osc filt env 2 copy WIP
Parts:
- removed J13: OscFiltEnv2Conn, Connector_PinHeader_2.54mm:PinHeader_1x10_P2.54mm_Vertical, symbol Connector_Generic:Conn_01x10
- removed J14: SubFiltEnv1Conn, Connector_PinHeader_2.54mm:PinHeader_1x10_P2.54mm_Vertical, symbol Connector_Generic:Conn_01x10
- removed J15: SubFiltEnv2Conn, Connector_PinHeader_2.54mm:PinHeader_1x10_P2.54mm_Vertical, symbol Connector_Generic:Conn_01x10
- removed RV11, RV12, RV13: 100K, Potentiometer_THT:Potentiometer_Piher_PT-6-V_Vertical, symbol Device:R_POT_TRIM_US
- removed U33: TL074, Package_DIP:DIP-14_W7.62mm, symbol Amplifier_Operational:TL074
- added C182, C183: 100nF, Capacitor_THT:C_Disc_D5.0mm_W2.5mm_P5.00mm, symbol Device:C_Small
- added J13, J15, J18: Conn_01x05, Connector_PinHeader_2.54mm:PinHeader_1x05_P2.54mm_Vertical, symbol Connector_Generic:Conn_01x05
- added J14, J19, J30: Conn_01x04, Connector_PinHeader_2.54mm:PinHeader_1x04_P2.54mm_Vertical, symbol Connector_Generic:Conn_01x04
- added U33, U50: TL072, Package_DIP:DIP-8_W7.62mm, symbol Amplifier_Operational:TL072
Connections:
- wire segments 3059 -> 3058
- no-connect marks 18 -> 15
Other:
- note removed: "Power for both envelopes"
- moved on the sheet: C100, C101, C106, C107, C110, C111, C112, C113, C88, C89, U13B, U14B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
