File: PCB/Boom-1/Boom-1.kicad_sch (KiCad schematic)
At the start: 702 parts, among them J27 PowerConn, J28 FV1Conn, J37 Osc1Conn, J38 Osc2Conn, J39 SubNoiseConn, J40 FiltConn2, J41 EnvGenConn2, J42 EnvGenConn1, J43 FXConn1, J44 FiltConn1, J45 FXConn2, J46 EnvGenConn3, Q1 2N3904, SW1 SW_DIP_x04, U1 CEM3340, U10 AS3320, U11 AS3310, U12 AS3310, U13 AS3310, U14 AS3310, U15 V2164D, U16 AS3310, U17 AS3310, U18 V2164D, U19 TL074, U2 CEM3340, U20 TL074, U21 TL072, U22 TL074, U23 TL074, U24 TL072, U25 TL074, U26 TL074, U27 TL072, U28 TL074, U29 TL072, U3 4013, U30 TL072, U31 TL072, U32 TL074, U33 TL072, U34 TL074, U35 TL072, U36 TL074, U37 TL074, U38 TL072, U39 TL074, U4 NOISE, U40 TL072, U41 TL074, U42 TL074, U43 TL072, U44 TL074, U45 L7905, U46 L7805, U47 TL072, U48 TL072, U49 TL072, U5 V2164D, U50 TL072, U51 TL072, U6 V2164D, U7 V2164D, U8 AS3320, U9 AS3320

Commit message: more wire unwrangling
Parts:
- C108, C109, C3, C31, C8, C87: symbol Device:CP_Small -> Device:C_Polarized_Small
- C152, C153, C154, C155: symbol Device:CP1_Small -> Device:C_Polarized_Small_US
- D1: symbol Device:D_Small_ALT -> Device:D_Small_Filled
- D3, D4, D5, D6: symbol Device:D_Zener_ALT -> Device:D_Zener_Filled
- RV1, RV16, RV18, RV2, RV3, RV4, RV6, RV7, RV8, RV9: symbol Device:R_POT_TRIM_US -> Device:R_Potentiometer_Trim_US
- RV17, RV19, RV20, RV5: symbol Device:R_POT_US -> Device:R_Potentiometer_US
Other:
- moved on the sheet: C53, R141, U31A

Commit message: way more untangling done; first chunk split
Connections:
- net OscFiltEnv2AmtWiper is gone; now on net OscFiltEnv1AmtWiper: J42.10 (Pin_10), R154.1, R155.1
- net OscAmpEnv_Gate: now reaches R267.1, U16.4 (GATE), U35.6 (-), U35.7
- net OscAmpEnv_Trig: now reaches C122.2, U35.1, U35.2 (-)
- net OscFiltEnv1_VCS: now reaches R178.1, U11.9 (VCS)
- net OscFiltEnv1_VCR: now reaches R173.1, R176.1, U11.13 (VCR)
- net OscFiltEnv1_Gate: now reaches R148.1, U11.4 (GATE), U27.6 (-), U27.7
- net OscFiltEnv1_Trig: now reaches C61.2, U27.1, U27.2 (-)
- net OscFiltEnv2_Trig: now reaches C62.2, U29.1, U29.2 (-)
- net OscFiltEnv2_Gate: now reaches R149.1, U12.4 (GATE), U29.6 (-), U29.7
- net LeftOut: now reaches J28.13 (Pin_13), U43.3 (+)
- net RightOut: now reaches J28.14 (Pin_14), U43.5 (+)
- net OscFiltEnv1_VCD: now reaches R182.1, R192.1, U11.12 (VCD)
- net OscFiltEnv1_VCA: now reaches R183.1, R193.1, U11.15 (VCA)
- net SubFiltEnv2_Trig: now reaches C74.2, U50.1, U50.2 (-)
- net SubFiltEnv2_Gate: now reaches R160.1, U14.4 (GATE), U50.6 (-), U50.7
- net SubFiltEnv1_Trig: now reaches C73.2, U33.1, U33.2 (-)
- net SubFiltEnv1_Gate: now reaches R159.1, U13.4 (GATE), U33.6 (-), U33.7
- net SubAmpEnv_Gate: now reaches R268.1, U17.4 (GATE), U40.6 (-), U40.7
- net SubAmpEnv_Trig: now reaches C123.2, U40.1, U40.2 (-)
- net LeftIn: now reaches J28.10 (Pin_10), RV18.2
- net RightIn: now reaches J28.11 (Pin_11), RV16.2
- net SEL0: now reaches J28.4 (Pin_4), SW1.8
- net SEL1: now reaches J28.5 (Pin_5), SW1.7
- net SEL2: now reaches J28.6 (Pin_6), SW1.6
- net SRC: now reaches J28.7 (Pin_7), SW1.5
- net IN_{2}: now reaches R143.1, R161.2, R175.2, U10.2 (IN2)
- net IN_{3}: now reaches R144.2, R163.2, R166.1, U10.17 (IN3)
- net Cap_{2}: now reaches C63.1, U10.4 (CAP2)
- net Cap_{3}: now reaches C60.1, U10.16 (CAP3)
- net Cap_{4}: now reaches C64.1, U10.11 (CAP4)
- net IN_{4}: now reaches R145.1, R162.1, R167.1, U10.18 (IN4)
- net Cap_{1}: now reaches C59.2, U10.5 (CAP1)
- net OscFiltEnv2_VCD: now reaches R184.1, R194.1, U12.12 (VCD)
- net OscFiltEnv2_VCR: now reaches R174.1, R177.1, U12.13 (VCR)
- net OscFiltEnv2_VCA: now reaches R185.1, R195.1, U12.15 (VCA)
- net OscFiltEnv2_VCS: now reaches R179.1, U12.9 (VCS)
- net SubFiltEnv1_VCD: now reaches R210.1, R220.1, U13.12 (VCD)
- net SubFiltEnv1_VCR: now reaches R188.1, R196.1, U13.13 (VCR)
- net SubFiltEnv1_VCA: now reaches R211.1, R221.1, U13.15 (VCA)
- net SubFiltEnv1_VCS: now reaches R198.1, U13.9 (VCS)
- net SubFiltEnv2_VCD: now reaches R212.1, R222.1, U14.12 (VCD)
- net SubFiltEnv2_VCR: now reaches R189.1, R197.1, U14.13 (VCR)
- net SubFiltEnv2_VCA: now reaches R213.1, R223.1, U14.15 (VCA)
- net SubFiltEnv2_VCS: now reaches R199.1, U14.9 (VCS)
- net SubAmpEnv_VCD: now reaches R292.1, R297.1, U17.12 (VCD)
- net SubAmpEnv_VCR: now reaches R280.1, R283.1, U17.13 (VCR)
- net SubAmpEnv_VCA: now reaches R293.1, R298.1, U17.15 (VCA)
- net SubAmpEnv_VCS: now reaches R285.1, U17.9 (VCS)
- net OscAmpEnv_VCD: now reaches R289.1, R296.1, U16.12 (VCD)
- net OscAmpEnv_VCR: now reaches R276.1, R281.1, U16.13 (VCR)
- net OscAmpEnv_VCA: now reaches R288.1, R295.1, U16.15 (VCA)
- net OscAmpEnv_VCS: now reaches R282.1, U16.9 (VCS)
- net FV1ControlCommonHigh renamed +3V3
- no-connect marks 14 -> 13
Other:
- note added: "ADSR Envelope Generators"
- moved on the sheet: C1, C10, C100, C101, C102, C103, C104, C105, C106, C107, C108, C109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

Commit message: more splitting up
Connections:
- net SubOscWaveIn: now reaches C3.1, TP1.1, U48.6 (-), U48.7
- net NoiseToOsc2FiltMix: now reaches C53.1, R141.2, R369.1, U31.2 (-), U7.5 (Io2)
- net PostVCA2: now reaches C145.2, R307.2, R315.2, TP38.1, U38.1
- net NoiseToSubFiltMix: now reaches R370.1, U7.4 (Io1)
Other:
- note added: "Noise Generator with unity-gain buffers"
- note added: "Unused units"
- moved on the sheet: C12, C13, C130, C131, C134, C135, C136, C137, C144, C145, C15, C16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

Commit message: now fits onto A0
Connections:
- net NoiseToSubFiltMixCV is gone; now on net NoiseToOsc2FiltMixCV: J39.10 (Pin_10), R58.1
- net WhiteNoiseOut is gone; now on net NoiseToOsc2FiltMixCV: J39.8 (Pin_8), R32.2, TP7.1, U25.1
- net OscFiltEnv1AmtWiper: no longer J42.10 (Pin_10), R154.1, R155.1
- net Freq_CV_In2: now reaches R11.1, R14.2, R16.1, R6.2, R8.1, U1.15 (Freq_CV_In)
- net Pulse_Wave2: now reaches R39.1, R51.2, U1.4 (Pulse_Wave)
- net Triangle_Wave2: now reaches R53.2, TP8.1, U1.10 (Triangle_Wave)
- net Osc1WaveMix: now reaches C51.2, R108.2, R109.2, R132.1, TP26.1, U21.7
- net Osc2FXPreSend: now reaches C54.1, R142.2, R366.2, R367.1, R370.2, R372.1, U30.2 (-), U5.5 (Io2)
- net FilterMix: now reaches R262.1, R263.2, R264.2, U49.2 (-)
- net Triangle_Wave: now reaches R45.2, TP2.1, U2.10 (Triangle_Wave), U48.5 (+)
- net Freq_CV_In: now reaches R10.1, R2.2, R3.1, R5.1, R7.2, U2.15 (Freq_CV_In)
- net Pulse_Wave: now reaches R29.1, R43.2, U2.4 (Pulse_Wave)
- net FiltMixSignal: now reaches R119.2, R120.2, R83.1, U24.1
- net SubOscWaveIn: no longer names the net of C3.1, TP1.1, U48.6 (-), U48.7
- new net OscFiltEnv2AmtWiper: J42.10 (Pin_10), R154.1, R155.1
Other:
- note added: "FIXME where is this supposed to go?"
- note added: "Wave creation"
- moved on the sheet: C1, C10, C102, C103, C104, C105, C108, C109, C11, C12, C128, C129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
