File: PCB/Boom-1-Top/Boom-1-Top.kicad_pcb (KiCad board)
At the start: 2 copper layers, 345 x 165 mm, 493 parts, among them J1 DEBUG, J10 MCLRCap, J10 PIC_DEBUG, J11 MCLRCap, J11 PIC_DEBUG, J12 MCLRCap, J12 PIC_DEBUG, J13 MCLRCap, J13 PIC_DEBUG, J14 MCLRCap, J14 PIC_DEBUG, J2 MIDI IN, J3 MIDI OUT, J37 Osc1Conn, J38 Osc2Conn, J39 SubNoiseConn, J4 MCLRCap, J4 PIC_DEBUG, J40 FiltConn2, J41 EnvGenConn2, J42 EnvGenConn1, J43 FXConn1, J44 FiltConn1, J45 FXConn2, J46 EnvGenConn3, J5 MCLRCap, J5 PIC_DEBUG, J6 MCLRCap, J6 PIC_DEBUG, J7 MCLRCap, J7 PIC_DEBUG, J8 MCLRCap, J8 PIC_DEBUG, J9 MCLRCap, J9 PIC_DEBUG, SW1 Rotary_Encoder, SW10 Rotary_Encoder, SW11 Rotary_Encoder, SW12 Rotary_Encoder, SW13 Rotary_Encoder, SW14 Rotary_Encoder, SW15 Rotary_Encoder_Switch, SW16 Rotary_Encoder_Switch, SW17 Rotary_Encoder, SW18 Rotary_Encoder, SW19 Rotary_Encoder, SW2 Rotary_Encoder, SW20 Rotary_Encoder, SW21 Rotary_Encoder, SW22 Rotary_Encoder, SW23 Rotary_Encoder, SW24 Rotary_Encoder, SW25 Rotary_Encoder, SW26 Rotary_Encoder, SW27 Rotary_Encoder, SW28 Rotary_Encoder_Switch, SW29 Rotary_Encoder, SW3 Rotary_Encoder, SW30 Rotary_Encoder, SW31 Rotary_Encoder, SW32 Rotary_Encoder, SW33 Rotary_Encoder, SW34 Rotary_Encoder, SW35 Rotary_Encoder, SW36 Rotary_Encoder, SW37 Rotary_Encoder, SW38 Rotary_Encoder, SW39 Rotary_Encoder, SW4 Rotary_Encoder, SW40 Rotary_Encoder, SW41 Reset, SW42 Reset, SW43 Reset, SW44 Reset, SW45 Reset, SW46 Reset, SW47 Reset, SW48 Reset, SW49 Reset, SW5 Rotary_Encoder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

Commit message: Updated STM32 config for MIDI and Bluetooth module
Parts:
- removed the C117 at (547.0, 322.2)
- removed the C118 at (524.8, 346.5)
- removed the C119 at (547.0, 324.7)
- removed the C123 at (551.0, 322.2)
- removed the C124 at (542.0, 331.9)
- removed the C127 at (560.3, 314.9)
- removed the C128 at (522.8, 351.7)
- removed the C131 at (538.9, 337.8)
- removed the C133 at (555.1, 320.0)
- removed the C134 at (530.2, 345.3)
- removed the C137 at (564.3, 312.4)
- removed C15, C16, C17, C18: 47nF, Capacitor_SMD:C_0603_1608Metric
- removed the J10 at (526.5, 335.6)
- removed the J11 at (537.7, 322.0)
- removed the J12 at (516.0, 344.1)
- removed the J13 at (408.0, 350.5)
- removed the J13 at (542.7, 313.5)
- removed the J14 at (533.0, 322.0)
- removed the J4 at (520.6, 340.3)
- removed the J5 at (417.2, 365.3)
- removed the J5 at (552.0, 313.5)
- removed the J6 at (412.6, 365.3)
- removed the J6 at (537.7, 329.2)
- removed the J7 at (542.7, 320.7)
- removed the J8 at (533.0, 329.2)
- removed the J9 at (547.3, 313.5)
- removed the R172 at (563.0, 322.5)
- removed the R173 at (568.3, 317.5)
- removed the R174 at (558.0, 327.5)
- removed the R175 at (550.9, 334.8)
- removed the R176 at (546.9, 339.8)
- removed the R177 at (542.2, 344.4)
- removed the R178 at (567.1, 320.0)
- removed the R179 at (538.8, 347.8)
- removed the R180 at (554.9, 330.0)
- removed the R181 at (554.9, 332.5)
- removed the R182 at (563.0, 325.0)
- removed R187, R19, R190, R191, R193, R20, R25, R26, R33, R34, R35, R36: 10K, Resistor_SMD:R_0603_1608Metric
- removed R188, R189, R192: 470R, Resistor_SMD:R_0603_1608Metric
- removed SW8, SW9: Rotary_Encoder, PEC11R:PEC11R-4x15F-N0024
- removed the U3 at (393.2, 321.6)
- removed the U4 at (400.6, 321.4)
- added C139: 47nF, Capacitor_SMD:C_0603_1608Metric, F.Cu at (64.0, 20.5)
- added C140: 47nF, Capacitor_SMD:C_0603_1608Metric, F.Cu at (56.8, 17.4)
- added J13: PIC_DEBUG, Connector_PinSocket_2.54mm:PinSocket_1x05_P2.54mm_Vertical, F.Cu at (298.0, 140.0)
- added J15: USB_B_Micro, Connector_USB:USB_Micro-B_Amphenol_10118194_Horizontal, F.Cu at (189.5, 35.0)
- added J16: SD_Card, Connector_Card:SD_Kyocera_145638009211859+, F.Cu at (231.5, 43.5)
- added J5: PIC_DEBUG, Connector_PinSocket_2.54mm:PinSocket_1x05_P2.54mm_Vertical, F.Cu at (72.0, 64.0)
- added J6: PIC_DEBUG, Connector_PinSocket_2.54mm:PinSocket_1x05_P2.54mm_Vertical, F.Cu at (74.5, 163.0)
- added SW53: Osc1TuneEncoder, PEC11R:PEC11R-4x15F-S0024, F.Cu at (72.5, 44.5)
- added U23: BLUENRG-M2SA, BLUENRG:XCVR_BLUENRG-M2SA, F.Cu at (369.0, 41.0)
- R183, R186: value 470R -> 10K
- SW1: value Rotary_Encoder -> Osc1SawEncoder
- SW2, SW4: value Rotary_Encoder -> Rotary_Encoder_Switch; footprint PEC11R:PEC11R-4x15F-N0024 -> PEC11R:PEC11R-4x15F-S0024
- SW41, SW42, SW43, SW44, SW45, SW46, SW47, SW48, SW49, SW50, SW51, SW52: footprint Button_Switch_THT:SW_PUSH_6mm -> PTS636:PTS636
- moved R185 590.2 mm to (56.8, 19.9)
- moved R186 587.8 mm to (75.8, -0.32)
- moved R184 584.0 mm to (71.8, -0.32)
- moved R183 577.5 mm to (68.0, 20.5)
- moved U3 564.6 mm to (38.0, 42.5)
- moved U4 520.8 mm to (37.5, 125.0)
- moved SW43 469.4 mm to (64.5, 62.5)
- moved SW45 451.6 mm to (116.5, 40.5)
- moved J7 438.7 mm to (111.5, 42.0)
- moved SW42 437.9 mm to (69.5, 104.5)
- moved U13 424.8 mm to (120.5, 53.5)
- moved SW44 419.2 mm to (65.5, 161.5)
- moved U5 416.9 mm to (38.0, 52.0)
- moved J4 408.1 mm to (77.5, 105.0)
- moved SW47 405.7 mm to (180.0, 49.5)
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Connections:
- net Net-(U1-Pad65) renamed SDIO_D0
- net Net-(U1-Pad66) renamed SDIO_D1
- net Net-(U1-Pad78) renamed SDIO_D2
- net Net-(U1-Pad79) renamed SDIO_D3
- net Net-(U1-Pad80) renamed SDIO_CLK
- net Net-(U1-Pad83) renamed SDIO_CMD
- R183 pad 1: Net-(J10-Pad1) -> +5V
- R184 pad 1: Net-(J9-Pad1) -> Net-(C139-Pad1)
- R184 pad 2: +5V -> Net-(R183-Pad2)
- R185 pad 1: Net-(J10-Pad1) -> Net-(R185-Pad1)
- R185 pad 2: +5V -> Net-(C140-Pad2)
- R186 pad 1: Net-(J11-Pad1) -> Net-(R185-Pad1)
- R186 pad 2: Net-(R186-Pad2) -> +5V
- U1 pad 55: SubAmpEnvGate -> Net-(U1-Pad55)
- U1 pad 56: SubAmpEnvTrigger -> Net-(U1-Pad56)
- U1 pad 57: OscFiltEnv2Gate -> Net-(U1-Pad57)
- U1 pad 58: OscFiltEnv2Trigger -> Net-(U1-Pad58)
- U1 pad 59: OscFiltEnv1Gate -> Net-(U1-Pad59)
- U1 pad 60: OscFiltEnv1Trigger -> Net-(U1-Pad60)
- U11 pad 17: Net-(C9-Pad2) -> Net-(U11-Pad17)
- U11 pad 18: Net-(C10-Pad1) -> Net-(U11-Pad18)
- U11 pad 4: Net-(C17-Pad2) -> Net-(C9-Pad2)
- U11 pad 5: Net-(C18-Pad1) -> Net-(C10-Pad1)
- U11 pad 9: Net-(U11-Pad9) -> Net-(SW4-PadS2)
- U13 pad 17: Net-(U13-Pad17) -> Net-(C140-Pad2)
- U13 pad 18: Net-(U13-Pad18) -> Net-(C139-Pad1)
Routing:
- added copper zone on B.Cu, net GND
- added copper zone on F.Cu, net GND
