File: PCB/Boom-1-Top/Boom-1-Top.sch (KiCad schematic (older format))
At the start: 1025 parts, among them J1 DEBUG, J10 PIC_DEBUG, J11 PIC_DEBUG, J12 PIC_DEBUG, J13 PIC_DEBUG, J14 PIC_DEBUG, J15 USB_B_Micro, J16 SD_Card, J17 BT_DEBUG, J18 12V Supply, J19 3V3 Bypass, J2 MIDI IN, J20 5V Bypass, J21 Env +12V Supply, J22 Env -12V Supply, J23 OLEDConn, J24 FiltConn1PassThru, J25 LeftI2C0Test, J26 AudioOutConn, J27 FiltConn2PassThru, J28 FiltConn2PassThruPower, J29 LeftI2C1Test, J3 MIDI OUT, J30 LeftI2C2Test, J31 LeftI2C3Test, J32 RightI2C0Test, J33 RightI2C1Test, J34 RightI2C2Test, J35 RightI2C3Test, J36 SPIBus1Test, J37 Osc1Conn, J38 Osc2Conn, J39 SubNoiseConn, J4 PIC_DEBUG, J40 FiltConn2, J41 EnvGenConn2, J42 EnvGenConn1, J43 FXConn1, J44 FiltConn1, J45 FXConn2, J46 EnvGenConn3, J47 BTTestConn, J48 MIDITestConn, J49 I2CBus1TestConn, J5 PIC_DEBUG, J50 I2CBus2TestConn, J51 OLEDTestConn, J52 SDIOTestConn, J53 HapticEngine, J6 PIC_DEBUG, J7 PIC_DEBUG, J8 PIC_DEBUG, J9 PIC_DEBUG, Q1 AO3401A, Q2 AO3401A, SW1 Osc1SawEncoder, SW10 SubToOsc2FiltEncoder, SW11 Osc1ToOsc2FiltEncoder, SW12 Osc1FiltFreqEncoder, SW13 Osc2FiltFreqEncoder, SW14 SubFiltFreqEncoder, SW15 OscFiltEnvAttackEncoder, SW16 SubFiltEnvAttackEncoder, SW17 Osc1FiltResEncoder, SW18 Osc2FiltResEncoder, SW19 SubFiltResEncoder, SW2 Osc1SqrEncoder, SW20 OscFiltEnvDecayEncoder, SW21 SubFiltEnvDecayEncoder, SW22 OscFiltEnvSustainEncoder, SW23 SubFiltEnvSustainEncoder, SW24 Osc1DriveEncoder, SW25 Osc2DistortionEncoder, SW26 OscFiltEnvReleaseEncoder, SW27 SubFiltEnvReleaseEncoder, SW28 FXWetDryEncoder, SW29 SubAmpEnvAttackEncoder, SW3 Rotary_Encoder, SW30 OscAmpEnvAttackEncoder, SW31 FXControl1Encoder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

Commit message: - Added EEPROM for fv1 - Feedback resistors for power supply
Parts:
- added R315: 9.53K, Resistor_SMD:R_0603_1608Metric, symbol Device:R_Small_US
- added U57: 24LC32, Package_DIP:DIP-8_W7.62mm_Socket, symbol Memory_EEPROM:24LC32
- R215: value 47K -> 49.9K
- R216: value 15K -> 16.2K
- R217: value 270R -> 49.9K
Connections:
- net +3V3: now also U57.8 (VCC)
- net +5V: now also R217.1
- net FV1EEpromSCL: now also U57.6 (SCL)
- net FV1EEpromSDA: now also U57.5 (SDA)
- net GND: now also R216.2, U57.1 (A0), U57.2 (A1), U57.3 (A2), U57.4 (GND), U57.7 (WP); no longer R217.2
- net at U42.3 (FB): now also R217.2, R315.1
Changed lines of the file:
@@
 P 6600 1650
 F 0 "R215" H 6668 1696 50  0000 L CNN
-F 1 "47K" H 6668 1605 50  0000 L CNN
+F 1 "49.9K" H 6668 1605 50  0000 L CNN
 F 2 "Resistor_SMD:R_0603_1608Metric" H 6600 1650 50  0001 C CNN
 F 3 "~" H 6600 1650 50  0001 C CNN
@@
 P 6600 1950
 F 0 "R216" H 6668 1996 50  0000 L CNN
-F 1 "15K" H 6668 1905 50  0000 L CNN
+F 1 "16.2K" H 6668 1905 50  0000 L CNN
 F 2 "Resistor_SMD:R_0603_1608Metric" H 6600 1950 50  0001 C CNN
 F 3 "~" H 6600 1950 50  0001 C CNN
@@
 $EndComp
 $Comp
-L Device:R_Small_US R217
-U 1 1 6498F374
-P 6600 2150
-F 0 "R217" H 6668 2196 50  0000 L CNN
-F 1 "270R" H 6668 2105 50  0000 L CNN
-F 2 "Resistor_SMD:R_0603_1608Metric" H 6600 2150 50  0001 C CNN
-F 3 "~" H 6600 2150 50  0001 C CNN
-	1    6600 2150
-	1    0    0    -1
-$EndComp
-$Comp
 L power:+3.3V #PWR0542
 U 1 1 649A05C2
@@
 L power:GND #PWR0543
 U 1 1 64B999A4
-P 6600 2250
-F 0 "#PWR0543" H 6600 2000 50  0001 C CNN
-F 1 "GND" H 6605 2077 50  0000 C CNN
-F 2 "" H 6600 2250 50  0001 C CNN
-F 3 "" H 6600 2250 50  0001 C CNN
-	1    6600 2250
+P 6600 2100
+F 0 "#PWR0543" H 6600 1850 50  0001 C CNN
+F 1 "GND" H 6605 1927 50  0000 C CNN
+F 2 "" H 6600 2100 50  0001 C CNN
+F 3 "" H 6600 2100 50  0001 C CNN
+	1    6600 2100
 	1    0    0    -1
 $EndComp
@@
 L power:GND #PWR0562
 U 1 1 61095109
-P 6600 3650
-F 0 "#PWR0562" H 6600 3400 50  0001 C CNN
-F 1 "GND" H 6605 3477 50  0000 C CNN
-F 2 "" H 6600 3650 50  0001 C CNN
-F 3 "" H 6600 3650 50  0001 C CNN
-	1    6600 3650
+P 6600 3500
+F 0 "#PWR0562" H 6600 3250 50  0001 C CNN
+F 1 "GND" H 6605 3327 50  0000 C CNN
+F 2 "" H 6600 3500 50  0001 C CNN
+F 3 "" H 6600 3500 50  0001 C CNN
+	1    6600 3500
 	1    0    0    -1
 $EndComp
@@
 Text GLabel 38150 42900 0    50   Input ~ 0
 LEFT_I2C_2_SDA
+Wire Wire Line
+	6600 2050 6600 2100
+$Comp
+L Device:R_Small_US R217
+U 1 1 60FE67FB
+P 6600 3050
+F 0 "R217" H 6668 3096 50  0000 L CNN
+F 1 "49.9K" H 6668 3005 50  0000 L CNN
+F 2 "Resistor_SMD:R_0603_1608Metric" H 6600 3050 50  0001 C CNN
+F 3 "~" H 6600 3050 50  0001 C CNN
+	1    6600 3050
+	1    0    0    -1
+$EndComp
+$Comp
+L Device:R_Small_US R315
+U 1 1 60FE6D34
+P 6600 3350
+F 0 "R315" H 6668 3396 50  0000 L CNN
+F 1 "9.53K" H 6668 3305 50  0000 L CNN
+F 2 "Resistor_SMD:R_0603_1608Metric" H 6600 3350 50  0001 C CNN
+F 3 "~" H 6600 3350 50  0001 C CNN
+	1    6600 3350
+	1    0    0    -1
+$EndComp
+$Comp
+L Memory_EEPROM:24LC32 U57
+U 1 1 616CDB8D
+P 34600 36100
+F 0 "U57" H 34600 36581 50  0000 C CNN
+F 1 "24LC32" H 34600 36490 50  0000 C CNN
+F 2 "Package_DIP:DIP-8_W7.62mm_Socket" H 34600 36100 50  0001 C CNN
+F 3 "http://ww1.microchip.com/downloads/en/DeviceDoc/21072G.pdf" H 34600 36100 50  0001 C CNN
+	1    34600 36100
+	1    0    0    -1
+$EndComp
+Text GLabel 35000 36000 2    50   Input ~ 0
+FV1EEpromSDA
+Text GLabel 35000 36100 2    50   Input ~ 0
+FV1EEpromSCL
+$Comp
+L power:+3.3V #PWR0989
+U 1 1 61C5C85F
+P 34600 35800
+F 0 "#PWR0989" H 34600 35650 50  0001 C CNN
+F 1 "+3.3V" V 34615 35928 50  0000 L CNN
+F 2 "" H 34600 35800 50  0001 C CNN
+F 3 "" H 34600 35800 50  0001 C CNN
+	1    34600 35800
+	0    1    1    0
+$EndComp
+$Comp
+L power:GND #PWR0990
+U 1 1 61C69018
+P 34600 36400
+F 0 "#PWR0990" H 34600 36150 50  0001 C CNN
+F 1 "GND" H 34605 36227 50  0000 C CNN
+F 2 "" H 34600 36400 50  0001 C CNN
+F 3 "" H 34600 36400 50  0001 C CNN
+	1    34600 36400
+	1    0    0    -1
+$EndComp
+$Comp
+L power:GND #PWR0991
+U 1 1 61C752B9
+P 34200 36000
+F 0 "#PWR0991" H 34200 35750 50  0001 C CNN
+F 1 "GND" V 34205 35872 50  0000 R CNN
+F 2 "" H 34200 36000 50  0001 C CNN
+F 3 "" H 34200 36000 50  0001 C CNN
+	1    34200 36000
+	0    1    1    0
+$EndComp
+$Comp
+L power:GND #PWR0992
+U 1 1 61C75725
+P 34200 36100
+F 0 "#PWR0992" H 34200 35850 50  0001 C CNN
+F 1 "GND" V 34205 35972 50  0000 R CNN
+F 2 "" H 34200 36100 50  0001 C CNN
+F 3 "" H 34200 36100 50  0001 C CNN
+	1    34200 36100
+	0    1    1    0
+$EndComp
+$Comp
+L power:GND #PWR0993
+U 1 1 61C75985
+P 34200 36200
+F 0 "#PWR0993" H 34200 35950 50  0001 C CNN
+F 1 "GND" V 34205 36072 50  0000 R CNN
+F 2 "" H 34200 36200 50  0001 C CNN
+F 3 "" H 34200 36200 50  0001 C CNN
+	1    34200 36200
+	0    1    1    0
+$EndComp
+$Comp
+L power:GND #PWR0994
+U 1 1 61C7A979
+P 35000 36200
+F 0 "#PWR0994" H 35000 35950 50  0001 C CNN
+F 1 "GND" V 35005 36072 50  0000 R CNN
+F 2 "" H 35000 36200 50  0001 C CNN
+F 3 "" H 35000 36200 50  0001 C CNN
+	1    35000 36200
+	0    -1   -1   0
+$EndComp
 $EndSCHEMATC

Commit message: - Added copper keepouts and dedicated ground plane for hse
Parts:
- R161: footprint Resistor_SMD:R_1206_3216Metric -> Resistor_SMD:R_0402_1005Metric
Changed lines of the file:
@@
 F 0 "R161" V 8995 6950 50  0000 C CNN
 F 1 "220R" V 9086 6950 50  0000 C CNN
-F 2 "Resistor_SMD:R_1206_3216Metric" H 9200 6950 50  0001 C CNN
+F 2 "Resistor_SMD:R_0402_1005Metric" H 9200 6950 50  0001 C CNN
 F 3 "~" H 9200 6950 50  0001 C CNN
 	1    9200 6950

Commit message: - Fixing 5VA power
Connections:
- net +12VA: no longer J40.8 (Pin_8)
- net -12VA: no longer J40.12 (Pin_12), J40.18 (Pin_18)
- net GND: no longer U56.6 (P1W)
- net GNDA: no longer J26.2 (Pin_2), J26.4 (Pin_4), J37.10 (Pin_10), J37.12 (Pin_12), J37.14 (Pin_14), J37.16 (Pin_16), J38.10 (Pin_10), J38.12 (Pin_12), J38.14 (Pin_14), J38.16 (Pin_16), J38.6 (Pin_6), J38.8 (Pin_8), J39.11 (Pin_11), J39.2 (Pin_2), J39.4 (Pin_4), J40.16 (Pin_16), J40.21 (Pin_21), J40.23 (Pin_23), J40.24 (Pin_24), J41.17 (Pin_17), J41.18 (Pin_18), J42.17 (Pin_17), J42.18 (Pin_18), J44.3 (Pin_3), J45.1 (Pin_1), J45.10 (Pin_10), J45.3 (Pin_3), J45.9 (Pin_9), J46.17 (Pin_17), J46.18 (Pin_18)
- net +5VA renamed +5VA_LEFT
- net +5VA_LEFT: no longer C114.1, C115.1, C116.1, C176.1, C178.1, C212.1, C232.1, C233.1, L4.2, L6.2, U10.3 (AVDD), U50.3 (AVDD), U8.3 (AVDD), U9.2 (ADDR0), U9.3 (AVDD)
- net Osc1HFTrackHigh: no longer names the net of J37.9 (Pin_9)
- net Osc1HFTrackWiper: no longer names the net of J37.11 (Pin_11)
- net Osc1HardSyncIn: no longer names the net of J37.15 (Pin_15)
- net Osc1SyncOut: no longer names the net of J37.13 (Pin_13)
- net Osc2HFTrackHigh: no longer names the net of J38.9 (Pin_9)
- net Osc2HFTrackWiper: no longer names the net of J38.11 (Pin_11)
- net Osc2HardSyncIn: no longer names the net of J38.15 (Pin_15)
- net Osc2SoftSyncIn: no longer names the net of J38.17 (Pin_17)
- net Osc2SyncOut: no longer names the net of J38.13 (Pin_13)
- net PinkNoiseOut: no longer names the net of J39.6 (Pin_6)
- net SubOct1Out: no longer names the net of J39.3 (Pin_3)
- net SubOct2Out: no longer names the net of J39.7 (Pin_7)
- net SubOctBothOut: no longer names the net of J39.5 (Pin_5)
- net WhiteNoiseOut: no longer names the net of J39.8 (Pin_8)
- new net +5VA_RIGHT: C114.1, C115.1, C116.1, C176.1, C178.1, L4.2, U10.3 (AVDD), U8.3 (AVDD), U9.2 (ADDR0), U9.3 (AVDD)
- new net +5VA_TOP: C212.1, C232.1, C233.1, L6.2, U50.3 (AVDD)
- new net MixOutGND: J26.2 (Pin_2), J26.4 (Pin_4), J45.10 (Pin_10)
- no-connect marks 26 -> 200
Other:
- moved on the sheet: C95, C99

Commit message: Zero ERC
Connections:
- net +12VA: no longer J24.1 (Pin_1), J28.12 (Pin_12), J28.3 (Pin_3), J28.6 (Pin_6), J28.9 (Pin_9), J40.14 (Pin_14), J40.2 (Pin_2), J44.1 (Pin_1)
- net -12VA: no longer J24.5 (Pin_5), J28.11 (Pin_11), J28.2 (Pin_2), J28.5 (Pin_5), J28.8 (Pin_8), J40.6 (Pin_6), J44.5 (Pin_5)
- net GND: now also R315.2
- net GNDA renamed FiltConn2GND
- net FiltConn2GND: no longer J24.3 (Pin_3), J24.7 (Pin_7), J44.7 (Pin_7)
- net L3B9: no longer names the net of U38.31 (OUT30)
- net L3G9: no longer names the net of U38.30 (OUT29)
- net L3R9: no longer names the net of U38.29 (OUT28)
- net L8B9: no longer names the net of U35.31 (OUT30)
- net L8G9: no longer names the net of U35.30 (OUT29)
- net L8R9: no longer names the net of U35.29 (OUT28)
- net Osc1SoftSyncIn: no longer names the net of J37.17 (Pin_17)
- new net FiltConn1+12V: J24.1 (Pin_1), J44.1 (Pin_1)
- new net FiltConn1-12V: J24.5 (Pin_5), J44.5 (Pin_5)
- new net FiltConn1-GND: J24.3 (Pin_3), J24.7 (Pin_7), J44.7 (Pin_7)
- new net FiltConn2+12V: J28.12 (Pin_12), J28.3 (Pin_3), J28.6 (Pin_6), J28.9 (Pin_9), J40.14 (Pin_14), J40.2 (Pin_2)
- new net FiltConn2-12V: J28.11 (Pin_11), J28.2 (Pin_2), J28.5 (Pin_5), J28.8 (Pin_8), J40.6 (Pin_6)
- no-connect marks 200 -> 334
