File: PCB/Boom-1-Top/Rotary_Encoders.kicad_sch (KiCad schematic)
At the start: 373 parts, among them J10 PIC_DEBUG, J11 PIC_DEBUG, J12 PIC_DEBUG, J13 PIC_DEBUG, J14 PIC_DEBUG, J4 PIC_DEBUG, J5 PIC_DEBUG, J6 PIC_DEBUG, J7 PIC_DEBUG, J8 PIC_DEBUG, J9 PIC_DEBUG, SW1 Osc1SawEncoder, SW10 SubToOsc2FiltEncoder, SW11 Osc1ToOsc2FiltEncoder, SW12 Osc1FiltFreqEncoder, SW13 Osc2FiltFreqEncoder, SW14 SubFiltFreqEncoder, SW15 OscFiltEnvAttackEncoder, SW16 SubFiltEnvAttackEncoder, SW17 Osc1FiltResEncoder, SW18 Osc2FiltResEncoder, SW19 SubFiltResEncoder, SW2 Osc1SqrEncoder, SW20 OscFiltEnvDecayEncoder, SW21 SubFiltEnvDecayEncoder, SW22 OscFiltEnvSustainEncoder, SW23 SubFiltEnvSustainEncoder, SW24 Osc1DriveEncoder, SW25 Osc2DistortionEncoder, SW26 OscFiltEnvReleaseEncoder, SW27 SubFiltEnvReleaseEncoder, SW28 FXWetDryEncoder, SW29 SubAmpEnvAttackEncoder, SW3 Rotary_Encoder, SW30 OscAmpEnvAttackEncoder, SW31 FXControl1Encoder, SW32 SubAmpEnvDecayEncoder, SW33 OscAmpEnvDecayEncoder, SW34 FXControl2Encoder, SW35 SubAmpEnvSustainEncoder, SW36 OscAmpEnvSustainEncoder, SW37 FXControl3Encoder, SW38 FXFeedbackEncoder, SW39 SubAmpEnvReleaseEncoder, SW4 Rotary_Encoder_Switch, SW40 OscAmpEnvReleaseEncoder, SW43 Reset, SW5 Rotary_Encoder, SW53 Osc1TuneEncoder, SW6 SubToSubFiltEncoder, SW7 SubNoiseEncoder, U11 PIC18F26Q43, U12 PIC18F26Q43, U13 PIC18F26Q43, U14 PIC18F26Q43, U15 PIC18F26Q43, U16 PIC18F26Q43, U17 PIC18F26Q43, U18 PIC18F26Q43, U19 PIC18F26Q43, U2 PIC18F26Q43, U20 PIC18F26Q43

Commit message: changed rotary encoder symbol to new one in the 5.99/6.x library
Parts:
- SW1, SW10, SW11, SW12, SW13, SW14, SW17, SW18, SW19, SW20, SW21, SW24, SW25, SW26, SW27, SW29, SW3, SW30, SW31, SW32, SW33, SW34, SW37, SW38, SW39, SW40, SW5, SW6, SW7: symbol Device:Rotary_Encoder -> Device:RotaryEncoder
- SW15, SW16, SW2, SW22, SW23, SW28, SW35, SW36, SW4, SW53: symbol Device:Rotary_Encoder_Switch -> Device:RotaryEncoder_Switch
Other:
- moved on the sheet: C1, C10, C11, C117, C118, C119, C12, C120, C121, C122, C123, C124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

Commit message: Top: Rotary Encoder cleanup, [WIP]
Connections:
- net FXWetDryEncoder_SW: now reaches SW28.S1, U14.9 (RA7/SW1)
- net at C21.2, R39.2: now also U2.18 (RC7/R4B); no longer U2.17 (RC6/R4A)
- net at C22.1, R40.1: now also U2.17 (RC6/R4A); no longer U2.18 (RC7/R4B)
Other:
- moved on the sheet: C1, C118, C120, C123, C124, C125, C126, C127, C128, C129, C130, C131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

Commit message: Top: finished first pass over the rotary encodes
Other:
- note added: "Left 0"
- note added: "Left 2"
- note added: "Left 3"
- note added: "Right 0"
- note added: "Right 1"
- moved on the sheet: C10, C11, C117, C119, C12, C121, C122, C124, C126, C127, C128, C129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

Commit message: Top: reworked & split Rotary Encoders a bit more ; grouped top-level misc parts for next split
Parts:
- removed C1, C10, C11, C12, C13, C139, C14, C140, C19, C2, C20, C21, C22, C23, C24, C25, C26, C27, C28, C29, C3, C30, C31, C32, C33, C34, C35, C36, C37, C38, C39, C4, C40, C41, C42, C43, C44, C45, C46, C47, C48, C49, C5, C50, C51, C52, C53, C54, C55, C56, C57, C58, C59, C6, C60, C61, C62, C63, C64, C65, C66, C67, C68, C69, C7, C70, C71, C72, C73, C74, C75, C76, C77, C78, C79, C8, C80, C9: 47nF, Capacitor_SMD:C_0603_1608Metric, symbol Device:C_Small
- removed C117, C118, C119, C120, C121, C122, C123, C124, C125, C126, C127, C128, C129, C130, C131, C132, C133, C134, C135, C136, C137, C138: 100nF, Capacitor_SMD:C_0402_1005Metric, symbol Device:C_Small
- removed D11, D14, D15, D17, D19, D23, D24, D25, D5, D6, D7, D9: B5819W, Diode_SMD:D_SOD-123, symbol Device:D_Small
- removed D12: Osc1SqrMixLED, LED_SMD:LED_0603_1608Metric, symbol Device:LED
- removed D13: Osc1SqrPWMLED, LED_SMD:LED_0603_1608Metric, symbol Device:LED
- removed D16: Osc2SqrMixLED, LED_SMD:LED_0603_1608Metric, symbol Device:LED
- removed D18: Osc2SqrPWMLED, LED_SMD:LED_0603_1608Metric, symbol Device:LED
- removed D43: OscFiltEnv1LED, LED_SMD:LED_0603_1608Metric, symbol Device:LED
- removed D44: OscFiltEnv2LED, LED_SMD:LED_0603_1608Metric, symbol Device:LED
- removed D52: OscFiltSusLED, LED_SMD:LED_0603_1608Metric, symbol Device:LED
- removed D53: OscFiltAmtLED, LED_SMD:LED_0603_1608Metric, symbol Device:LED
- removed D54: SubFilt1LED, LED_SMD:LED_0603_1608Metric, symbol Device:LED
- removed D55: SubFilt2LED, LED_SMD:LED_0603_1608Metric, symbol Device:LED
- removed D58: SubFiltSusLED, LED_SMD:LED_0603_1608Metric, symbol Device:LED
- removed D59: SubFiltAmtLED, LED_SMD:LED_0603_1608Metric, symbol Device:LED
- removed D62: OscAmpEnvSusLED, LED_SMD:LED_0603_1608Metric, symbol Device:LED
- removed D63: OscAmpEnvAmtLED, LED_SMD:LED_0603_1608Metric, symbol Device:LED
- removed D64: SubAmpEnvSusLED, LED_SMD:LED_0603_1608Metric, symbol Device:LED
- removed D65: SubAmpEnvAmtLED, LED_SMD:LED_0603_1608Metric, symbol Device:LED
- removed J10, J11, J12, J13, J14, J4, J5, J6, J7, J8, J9: PIC_DEBUG, Connector_PinHeader_1.27mm:PinHeader_1x05_P1.27mm_Vertical, symbol Connector_Generic:Conn_01x05
- removed R1, R10, R100, R101, R102, R103, R104, R105, R106, R107, R108, R109, R11, R110, R111, R112, R113, R114, R115, R116, R117, R118, R119, R12, R120, R121, R122, R123, R124, R125, R126, R127, R128, R129, R13, R130, R131, R132, R133, R134, R135, R136, R137, R138, R139, R14, R140, R141, R142, R143, R144, R145, R146, R147, R148, R149, R15, R150, R151, R152, R153, R154, R155, R156, R157, R158, R159, R16, R160, R17, R18, R183, R184, R185, R186, R2, R21, R22, R23, R24, R27, R28, R29, R3, R30, R31, R32, R37, R38, R39, R4, R40, R41, R42, R43, R44, R45, R46, R47, R48, R49, R5, R50, R51, R52, R53, R54, R55, R56, R57, R58, R59, R6, R60, R61, R62, R63, R64, R65, R66, R67, R68, R69, R7, R70, R71, R72, R73, R74, R75, R76, R77, R78, R79, R8, R80, R81, R82, R83, R84, R85, R86, R87, R88, R89, R9, R90, R91, R92, R93, R94, R95, R96, R97, R98, R99: 10K, Resistor_SMD:R_0402_1005Metric, symbol Device:R_Small_US
- removed R172, R173, R174, R175, R176, R177, R178, R179, R180, R181, R182: 10K, Resistor_SMD:R_0603_1608Metric, symbol Device:R_Small_US
- removed R276, R277, R278, R279, R280, R281, R282, R283, R284, R285, R286, R287, R288, R289, R290, R291: 42R2, Resistor_SMD:R_0603_1608Metric, symbol Device:R_Small_US
- removed SW1: Osc1SawEncoder, PEC11R:PEC11R-4x15F-N0024, symbol Device:RotaryEncoder
- removed SW10: SubToOsc2FiltEncoder, PEC11R:PEC11R-4x15F-N0024, symbol Device:RotaryEncoder
- removed SW11: Osc1ToOsc2FiltEncoder, PEC11R:PEC11R-4x15F-N0024, symbol Device:RotaryEncoder
- removed SW12: Osc1FiltFreqEncoder, PEC11R:PEC11R-4x15F-N0024, symbol Device:RotaryEncoder
- removed SW13: Osc2FiltFreqEncoder, PEC11R:PEC11R-4x15F-N0024, symbol Device:RotaryEncoder
- removed SW14: SubFiltFreqEncoder, PEC11R:PEC11R-4x15F-N0024, symbol Device:RotaryEncoder
- removed SW15: OscFiltEnvAttackEncoder, PEC11R:PEC11R-4x15F-S0024, symbol Device:RotaryEncoder_Switch
- removed SW16: SubFiltEnvAttackEncoder, PEC11R:PEC11R-4x15F-S0024, symbol Device:RotaryEncoder_Switch
- removed SW17: Osc1FiltResEncoder, PEC11R:PEC11R-4x15F-N0024, symbol Device:RotaryEncoder
- removed SW18: Osc2FiltResEncoder, PEC11R:PEC11R-4x15F-N0024, symbol Device:RotaryEncoder
- removed SW19: SubFiltResEncoder, PEC11R:PEC11R-4x15F-N0024, symbol Device:RotaryEncoder
- removed SW2: Osc1SqrEncoder, PEC11R:PEC11R-4x15F-S0024, symbol Device:RotaryEncoder_Switch
- removed SW20: OscFiltEnvDecayEncoder, PEC11R:PEC11R-4x15F-N0024, symbol Device:RotaryEncoder
- removed SW21: SubFiltEnvDecayEncoder, PEC11R:PEC11R-4x15F-N0024, symbol Device:RotaryEncoder
- removed SW22: OscFiltEnvSustainEncoder, PEC11R:PEC11R-4x15F-S0024, symbol Device:RotaryEncoder_Switch
- removed SW23: SubFiltEnvSustainEncoder, PEC11R:PEC11R-4x15F-S0024, symbol Device:RotaryEncoder_Switch
- removed SW24: Osc1DriveEncoder, PEC11R:PEC11R-4x15F-N0024, symbol Device:RotaryEncoder
- removed SW25: Osc2DistortionEncoder, PEC11R:PEC11R-4x15F-N0024, symbol Device:RotaryEncoder
- removed SW26: OscFiltEnvReleaseEncoder, PEC11R:PEC11R-4x15F-N0024, symbol Device:RotaryEncoder
- removed SW27: SubFiltEnvReleaseEncoder, PEC11R:PEC11R-4x15F-N0024, symbol Device:RotaryEncoder
- removed SW28: FXWetDryEncoder, PEC11R:PEC11R-4x15F-S0024, symbol Device:RotaryEncoder_Switch
- removed SW29: SubAmpEnvAttackEncoder, PEC11R:PEC11R-4x15F-N0024, symbol Device:RotaryEncoder
- removed SW3, SW5: Rotary_Encoder, PEC11R:PEC11R-4x15F-N0024, symbol Device:RotaryEncoder
- removed SW30: OscAmpEnvAttackEncoder, PEC11R:PEC11R-4x15F-N0024, symbol Device:RotaryEncoder
- removed SW31: FXControl1Encoder, PEC11R:PEC11R-4x15F-N0024, symbol Device:RotaryEncoder
- removed SW32: SubAmpEnvDecayEncoder, PEC11R:PEC11R-4x15F-N0024, symbol Device:RotaryEncoder
- removed SW33: OscAmpEnvDecayEncoder, PEC11R:PEC11R-4x15F-N0024, symbol Device:RotaryEncoder
- removed SW34: FXControl2Encoder, PEC11R:PEC11R-4x15F-N0024, symbol Device:RotaryEncoder
- removed SW35: SubAmpEnvSustainEncoder, PEC11R:PEC11R-4x15F-S0024, symbol Device:RotaryEncoder_Switch
- removed SW36: OscAmpEnvSustainEncoder, PEC11R:PEC11R-4x15F-S0024, symbol Device:RotaryEncoder_Switch
- removed SW37: FXControl3Encoder, PEC11R:PEC11R-4x15F-N0024, symbol Device:RotaryEncoder
- removed SW38: FXFeedbackEncoder, PEC11R:PEC11R-4x15F-N0024, symbol Device:RotaryEncoder
- removed SW39: SubAmpEnvReleaseEncoder, PEC11R:PEC11R-4x15F-N0024, symbol Device:RotaryEncoder
- removed SW4: Rotary_Encoder_Switch, PEC11R:PEC11R-4x15F-S0024, symbol Device:RotaryEncoder_Switch
- removed SW40: OscAmpEnvReleaseEncoder, PEC11R:PEC11R-4x15F-N0024, symbol Device:RotaryEncoder
- removed SW43: Reset, PTS636:PTS636, symbol Switch:SW_Push
- removed SW53: Osc1TuneEncoder, PEC11R:PEC11R-4x15F-S0024, symbol Device:RotaryEncoder_Switch
- removed SW6: SubToSubFiltEncoder, PEC11R:PEC11R-4x15F-N0024, symbol Device:RotaryEncoder
- removed SW7: SubNoiseEncoder, PEC11R:PEC11R-4x15F-N0024, symbol Device:RotaryEncoder
- removed U11, U12, U13, U14, U15, U16, U17, U18, U19, U2, U20: PIC18F26Q43, Package_SO:SSOP-28_5.3x10.2mm_P0.65mm, symbol PIC18F26Q43:PIC18F26Q43
Connections:
- no-connect marks 72 -> 0
Other:
- added sheet Left 0:000 (L0_000.kicad_sch)
- added sheet Left 0:001 (L0_001.kicad_sch)
- added sheet Left 0:010 (L0_010.kicad_sch)
- added sheet Left 0:011 (L0_011.kicad_sch)
- added sheet Left 0:100 (L0_100.kicad_sch)
- added sheet Left 2:000 (L2_000.kicad_sch)
- added sheet Left 2:001 (L2_001.kicad_sch)
- added sheet Left 3:000 (L3_000.kicad_sch)
- added sheet Right 0:000 (R0_000.kicad_sch)
- added sheet Right 1:000 (R1_000.kicad_sch)
- added sheet Right 1:001 (R1_001.kicad_sch)
- note removed: "GND"
- note removed: "LEFT0:000"
- note removed: "LEFT0:001"
- note removed: "LEFT0:010"
- note removed: "LEFT0:011"
- note removed: "LEFT0:100"
- note removed: "LEFT2:000"
- note removed: "LEFT2:001"
- note removed: "LEFT3:000"
- note removed: "Left 0"
- note removed: "Left 2"
- note removed: "Left 3"
- note removed: "PGC"
- note removed: "PGD"
- note removed: "RIGHT0:000"
- note removed: "RIGHT1:000"
- note removed: "RIGHT1:001"
- note removed: "Right 0"
- note removed: "Right 1"
- note removed: "VDD"
- note removed: "VPP/MCLR"
