File: PCB/Boom-1-Top/Boom-1-Top.kicad_sch (KiCad schematic)
At the start: 114 parts, among them J18 12V Supply, J21 Env +12V Supply, J22 Env -12V Supply, J24 FiltConn1PassThru, J26 AudioOutConn, J27 FiltConn2PassThru, J28 FiltConn2PassThruPower, J39 SubNoiseConn, J40 FiltConn2, J41 EnvGenConn2, J42 EnvGenConn1, J43 FXConn1, J44 FiltConn1, J45 FXConn2, J46 EnvGenConn3, U10 DAC7678xPW, U43 V2164D, U44 V2164D, U45 TL074, U46 TL074, U47 TL074, U5 DAC7678xPW, U50 DAC7678xPW, U55 MCP4651, U56 MCP4651, U57 24LC32, U6 DAC7678xPW, U7 DAC7678xPW, U8 DAC7678xPW, U9 DAC7678xPW

Commit message: Top: finished first pass over the rotary encodes
Other:
- moved on the sheet: C103, C104, C105, C106, C107, C108, C109, C110, C111, C112, C113, C114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

Commit message: Top: reworked & split Rotary Encoders a bit more ; grouped top-level misc parts for next split
Other:
- moved on the sheet: C103, C104, C105, C106, C107, C108, C109, C110, C111, C112, C113, C114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

Commit message: Top: moved power connectors to Power Rails; moved anything pertaining to DACs into DACs
Parts:
- removed C103, C176, C230, C232: 10uF, Capacitor_SMD:C_1206_3216Metric, symbol Device:C_Small
- removed C105: 100nF, Capacitor_SMD:C_0402_1005Metric, symbol Device:C_Small
- removed C106, C178, C231, C233: 10nF, Capacitor_SMD:C_0402_1005Metric, symbol Device:C_Small
- removed C108: 100nF, Capacitor_SMD:C_0402_1005Metric, symbol Device:CP_Small
- removed J18: 12V Supply, TerminalBlock:TerminalBlock_bornier-2_P5.08mm, symbol Connector:Screw_Terminal_01x02
- removed J21: Env +12V Supply, TerminalBlock:TerminalBlock_bornier-2_P5.08mm, symbol Connector:Screw_Terminal_01x02
- removed J22: Env -12V Supply, TerminalBlock:TerminalBlock_bornier-2_P5.08mm, symbol Connector:Screw_Terminal_01x02
- removed L3, L4, L5, L6: 39nH, Inductor_SMD:L_0402_1005Metric, symbol Device:L_Small
- removed U6: DAC7678xPW, Package_SO:TSSOP-16_4.4x5mm_P0.65mm, symbol DAC7678:DAC7678xPW
Connections:
- no-connect marks 54 -> 52
Other:
- note removed: "Analog Hump"
- note removed: "DAC_LEFT0:010"
- note removed: "Left Side of Board"
- note removed: "Right Side of Board"

Commit message: actually moved the DAC-related stuff; DAC page to A1, top-level to A4
Parts:
- removed C104, C109, C111, C112, C113, C181, C182, C183, C184, C185, C186, C205, C206, C207, C208, C211, C237, C238: 100nF, Capacitor_SMD:C_0402_1005Metric, symbol Device:C_Small
- removed C107, C110, C114, C115, C116, C212: 100nF, Capacitor_SMD:C_0402_1005Metric, symbol Device:CP_Small
- removed C189, C190, C191, C192, C193, C194: 560pF, Capacitor_SMD:C_0402_1005Metric, symbol Device:C_Small
- removed C197, C198, C199, C200, C201, C202: 100pF, Capacitor_SMD:C_0402_1005Metric, symbol Device:C_Small
- removed D10, D8: B5819W, Diode_SMD:D_SOD-123, symbol Device:D_Schottky_Small
- removed J24: FiltConn1PassThru, Connector_PinSocket_2.54mm:PinSocket_2x04_P2.54mm_Vertical, symbol Connector_Generic:Conn_02x04_Odd_Even
- removed J26: AudioOutConn, Connector_PinSocket_2.54mm:PinSocket_2x02_P2.54mm_Vertical, symbol Connector_Generic:Conn_02x02_Odd_Even
- removed J27: FiltConn2PassThru, Connector_PinSocket_2.54mm:PinSocket_1x08_P2.54mm_Vertical, symbol Connector_Generic:Conn_01x08
- removed J28: FiltConn2PassThruPower, Connector_PinSocket_2.54mm:PinSocket_1x12_P2.54mm_Vertical, symbol Connector_Generic:Conn_01x12
- removed J39: SubNoiseConn, Connector_PinHeader_2.54mm:PinHeader_2x06_P2.54mm_Vertical, symbol Connector_Generic:Conn_02x06_Odd_Even
- removed J40: FiltConn2, Connector_PinHeader_2.54mm:PinHeader_2x12_P2.54mm_Vertical, symbol Connector_Generic:Conn_02x12_Odd_Even
- removed J41: EnvGenConn2, Connector_PinHeader_2.54mm:PinHeader_2x09_P2.54mm_Vertical, symbol Connector_Generic:Conn_02x09_Odd_Even
- removed J42: EnvGenConn1, Connector_PinHeader_2.54mm:PinHeader_2x09_P2.54mm_Vertical, symbol Connector_Generic:Conn_02x09_Odd_Even
- removed J43: FXConn1, Connector_PinHeader_2.54mm:PinHeader_2x08_P2.54mm_Vertical, symbol Connector_Generic:Conn_02x08_Odd_Even
- removed J44: FiltConn1, Connector_PinHeader_2.54mm:PinHeader_2x04_P2.54mm_Vertical, symbol Connector_Generic:Conn_02x04_Odd_Even
- removed J45: FXConn2, Connector_PinHeader_2.54mm:PinHeader_2x05_P2.54mm_Vertical, symbol Connector_Generic:Conn_02x05_Odd_Even
- removed J46: EnvGenConn3, Connector_PinHeader_2.54mm:PinHeader_2x09_P2.54mm_Vertical, symbol Connector_Generic:Conn_02x09_Odd_Even
- removed R222, R223, R226, R227, R228, R229, R230, R231, R234, R235, R236, R237, R238, R239, R242, R243, R244, R245, R254, R255, R256, R257, R258, R259: 30K, Resistor_SMD:R_0805_2012Metric, symbol Device:R_Small_US
- removed R246, R247, R248, R249, R250, R251: 510R, Resistor_SMD:R_0805_2012Metric, symbol Device:R_Small_US
- removed R262, R263: 7.5K, Resistor_SMD:R_0805_2012Metric, symbol Device:R_Small_US
- removed U10, U5, U50, U7, U8, U9: DAC7678xPW, Package_SO:TSSOP-16_4.4x5mm_P0.65mm, symbol DAC7678:DAC7678xPW
- removed U43, U44: V2164D, Package_SO:SOIC-16_3.9x9.9mm_P1.27mm, symbol CustomSymbols:V2164D
- removed U45, U46, U47: TL074, Package_SO:SOIC-14_3.9x8.7mm_P1.27mm, symbol Amplifier_Operational:TL074
- removed U55, U56: MCP4651, Package_SO:TSSOP-14_4.4x5mm_P0.65mm, symbol MCP4651:MCP4651
- removed U57: 24LC32, Package_DIP:DIP-8_W7.62mm_Socket, symbol Memory_EEPROM:24LC32
Connections:
- no-connect marks 52 -> 0
Other:
- note removed: "DAC_LEFT0:000"
- note removed: "DAC_LEFT0:100"
- note removed: "DAC_LEFT2:000"
- note removed: "DAC_RIGHT2:000"
- note removed: "DAC_RIGHT2:010"
- note removed: "DAC_RIGHT2:100"
