File: PCB/Boom-1-Top/DACs.kicad_sch (KiCad schematic)
At the start: 46 parts, among them J24 FiltConn1PassThru, J26 AudioOutConn, J27 FiltConn2PassThru, J28 FiltConn2PassThruPower, J36 SPIBus1Test, J37 Osc1Conn, J38 Osc2Conn, J39 SubNoiseConn, J40 FiltConn2, J41 EnvGenConn2, J42 EnvGenConn1, J43 FXConn1, J44 FiltConn1, J46 EnvGenConn3, U10 DAC7678xPW, U3 AD5290, U4 AD5290, U5 DAC7678xPW, U55 MCP4651, U56 MCP4651, U6 DAC7678xPW, U7 DAC7678xPW, U8 DAC7678xPW, U9 DAC7678xPW

Commit message: Top: done splitting up the DAC-related parts
Parts:
- removed J26: AudioOutConn, Connector_PinSocket_2.54mm:PinSocket_2x02_P2.54mm_Vertical, symbol Connector_Generic:Conn_02x02_Odd_Even
Other:
- moved on the sheet: C101, C102, C104, C105, C107, C108, C109, C110, C111, C112, C113, C114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
